File: Diseño_PCB/SmartWatch/SmartWatch.kicad_pcb (KiCad board)
At the start: 2 copper layers, 45 x 45 mm, 27 parts, among them J1 Input_BAT, J2 USB_B_Micro, J3 FTDI, SW1 SW_SPST, SW2 SW_Push, SW3 SW_Push, SW4 SW_Push_Dual, SW5 SW_Push_Dual, SW6 SW_Push_Dual, U1 TP4056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

Commit message: Actualizacion del PCB final
Routing:
- net GND: track 127.2 -> 128.2 mm
Changed lines of the file:
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@@
     (pad "4" thru_hole oval (at 4 -10.6 90) (size 2 2) (drill 1) (layers "*.Cu" "*.Mask")
       (net 20 "/SDA") (pinfunction "SDA") (pintype "input"))
-    (model "D:/APPS Mauri/KiCad Carpetas/EESTN5 - Librerias Kicad/EESTN5.3dshapes/128x64_I2C_OLEDDisplay_Adafruit.wrl"
+    (model "D:/APPS Mauri/KiCad Carpetas/EESTN5 - Librerias Kicad/EESTN5.3dshapes/128x64_I2C_OLEDDisplay_Adafruit.wrl" hide
       (offset (xyz 0 0 -7.5))
+      (scale (xyz 1 1 1))
+      (rotate (xyz 0 0 0))
+    )
+    (model "C:/Users/estudiante/Documents/Kicad_Archivos/Librerias-Kicad-master/EESTN5.3dshapes/128x64_I2C_OLEDDisplay_Adafruit.wrl"
+      (offset (xyz 0 0 -6.5))
       (scale (xyz 1 1 1))
       (rotate (xyz 0 0 0))
@@
   (segment (start 153.83 97.21) (end 157.245 100.625) (width 0.75) (layer "F.Cu") (net 1))
   (segment (start 155.15 90.41) (end 153.83 91.73) (width 0.75) (layer "F.Cu") (net 1))
+  (segment (start 190.59 102.07) (end 166.914998 102.07) (width 0.75) (layer "F.Cu") (net 1))
+  (segment (start 190.99 101.67) (end 190.59 102.07) (width 0.75) (layer "F.Cu") (net 1))
   (segment (start 157.245 100.625) (end 165.469998 100.625) (width 0.75) (layer "F.Cu") (net 1))
   (segment (start 191.5125 97.96) (end 190.99 98.4825) (width 0.75) (layer "F.Cu") (net 1))
   (segment (start 153.83 91.73) (end 153.83 97.21) (width 0.75) (layer "F.Cu") (net 1))
-  (segment (start 188.82 102.07) (end 166.914998 102.07) (width 0.75) (layer "F.Cu") (net 1))
-  (segment (start 190.99 99.9) (end 188.82 102.07) (width 0.75) (layer "F.Cu") (net 1))
+  (segment (start 190.99 99.9) (end 190.99 101.67) (width 0.75) (layer "F.Cu") (net 1))
+  (segment (start 166.914998 102.07) (end 165.469998 100.625) (width 0.75) (layer "F.Cu") (net 1))
   (segment (start 190.99 98.4825) (end 190.99 99.9) (width 0.75) (layer "F.Cu") (net 1))
   (segment (start 191.5125 96.675) (end 191.5125 97.96) (width 0.75) (layer "F.Cu") (net 1))
   (segment (start 160.18 90.41) (end 155.15 90.41) (width 0.75) (layer "F.Cu") (net 1))
-  (segment (start 166.914998 102.07) (end 165.469998 100.625) (width 0.75) (layer "F.Cu") (net 1))
   (via (at 160.18 90.41) (size 2) (drill 0.4) (layers "F.Cu" "B.Cu") (net 1))
   (via (at 165.469998 100.625) (size 2) (drill 0.4) (layers "F.Cu" "B.Cu") (net 1))

Commit message: Arreglo PCB, Creacion de la carcasa 3D
Changed lines of the file:
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@@
     (pad_to_mask_clearance 0)
     (pcbplotparams
-      (layerselection 0x0000000_7fffffff)
+      (layerselection 0x0000000_fffffffe)
       (plot_on_all_layers_selection 0x0001000_00000000)
       (disableapertmacros false)
@@
       (subtractmaskfromsilk false)
       (outputformat 5)
-      (mirror true)
+      (mirror false)
       (drillshape 1)
       (scaleselection 1)
@@
     (fp_line (start 10.04 7.3) (end 10.04 7.94)
       (stroke (width 0.1) (type solid)) (layer "F.Fab"))
-    (pad "1" thru_hole rect (at 0 0 270) (size 1.7 1.7) (drill 1) (layers "*.Cu" "*.Mask")
+    (pad "1" thru_hole rect (at 0 0 270) (size 2 2) (drill 1) (layers "*.Cu" "*.Mask")
       (net 1 "GND") (pinfunction "Pin_1") (pintype "passive"))
-    (pad "2" thru_hole oval (at 0 2.54 270) (size 1.7 1.7) (drill 1) (layers "*.Cu" "*.Mask")
+    (pad "2" thru_hole oval (at 0 2.54 270) (size 2 2) (drill 1) (layers "*.Cu" "*.Mask")
       (net 2 "+3.3V") (pinfunction "Pin_2") (pintype "passive"))
-    (pad "3" thru_hole oval (at 0 5.08 270) (size 1.7 1.7) (drill 1) (layers "*.Cu" "*.Mask")
+    (pad "3" thru_hole oval (at 0 5.08 270) (size 2 2) (drill 1) (layers "*.Cu" "*.Mask")
       (net 22 "/Rx") (pinfunction "Pin_3") (pintype "passive"))
-    (pad "4" thru_hole oval (at 0 7.62 270) (size 1.7 1.7) (drill 1) (layers "*.Cu" "*.Mask")
+    (pad "4" thru_hole oval (at 0 7.62 270) (size 2 2) (drill 1) (layers "*.Cu" "*.Mask")
       (net 23 "/Tx") (pinfunction "Pin_4") (pintype "passive"))
     (model "${KICAD6_3DMODEL_DIR}/Connector_PinHeader_2.54mm.3dshapes/PinHeader_1x04_P2.54mm_Horizontal.wrl" hide
